Commit message: iiwa dependency fix and initial plate

File: robot_agent_gazebo/models/kuka_with_plate/urdf/EEplate.urdf.xacro (robot description, xacro)
@@ -3,5 +3,5 @@
 <robot xmlns:xacro="http://www.ros.org/wiki/xacro">
 	<xacro:macro name="EEplate" params="parent name radius thickness *origin">
-		<joint name="${parent}_${name}_plate_joint" type="fixed">
+		<joint name="${parent}_${name}_joint" type="fixed">
 			<xacro:insert_block name="origin"/>
 			<parent link="${parent}"/>
@@ -9,10 +9,6 @@
 		</joint>
 		<link name="${name}_base">
-			<inertial>
-				<mass value="0.1"/>
-				<inertia ixx="0.4" ixy="0.0" ixz="0.0" iyy="0.4" iyz="0.0" izz="0.2"/>
-			</inertial>
 			<visual>
-				<origin xyz="0 0 ${thickness}*0.5" rpy="0 0 0"/>
+				<origin xyz="${-radius} 0 0" rpy="0 0 0"/>
 				<geometry>
 					<cylinder radius="${radius}" length="${thickness}"/>
@@ -20,5 +16,5 @@
 			</visual>
 			<collision>
-				<origin xyz="0 0 ${thickness}*0.5" rpy="0 0 0"/>
+				<origin xyz="${-radius} 0 0" rpy="0 0 0"/>
 				<geometry>
 					<cylinder radius="${radius}" length="${thickness}"/>

File: robot_agent_gazebo/models/kuka_with_plate/urdf/iiwa7.urdf.xacro (robot description, xacro)
@@ -2,7 +2,7 @@
 <robot name="iiwa7" xmlns:xacro="http://www.ros.org/wiki/xacro">
   <!-- Import Rviz colors -->
-  <xacro:include filename="$(find iiwa_description)/urdf/materials.xacro" />
+  <xacro:include filename="$(find robot_agent_gazebo)/models/kuka_with_plate/urdf/materials.xacro" />
   <!--Import the lbr iiwa macro -->
-  <xacro:include filename="$(find iiwa_description)/urdf/iiwa7.xacro"/>
+  <xacro:include filename="$(find robot_agent_gazebo)/models/kuka_with_plate/urdf/iiwa7.xacro"/>
   <xacro:arg name="hardware_interface" default="EffortJointInterface"/>
   <xacro:arg name="robot_name" default="iiwa"/>

File: robot_agent_gazebo/models/kuka_with_plate/urdf/iiwa7.xacro (robot description, xacro)
@@ -2,9 +2,9 @@
 <robot xmlns:xacro="http://www.ros.org/wiki/xacro">
   <!-- Import all Gazebo-customization elements, including Gazebo colors -->
-  <xacro:include filename="$(find iiwa_description)/urdf/iiwa.gazebo.xacro" />
+  <xacro:include filename="$(find robot_agent_gazebo)/models/kuka_with_plate/urdf/iiwa.gazebo.xacro" />
   <!-- Import Transmissions -->
-  <xacro:include filename="$(find iiwa_description)/urdf/iiwa.transmission.xacro" />
+  <xacro:include filename="$(find robot_agent_gazebo)/models/kuka_with_plate/urdf/iiwa.transmission.xacro" />
   <!-- Include Utilities -->
-  <xacro:include filename="$(find iiwa_description)/urdf/utilities.xacro" />
+  <xacro:include filename="$(find robot_agent_gazebo)/models/kuka_with_plate/urdf/utilities.xacro" />
   <!-- some constants -->
   <xacro:property name="safety_controller_k_pos" value="100" />
@@ -29,12 +29,12 @@
         <origin xyz="0 0 0" rpy="0 0 0"/>
         <geometry>
-          <mesh filename="package://iiwa_description/meshes/iiwa7/visual/link_0.stl"/>
-        </geometry>
-        <material name="Grey"/>
-      </visual>
-      <collision>
-        <origin xyz="0 0 0" rpy="0 0 0"/>
-        <geometry>
-          <mesh filename="package://iiwa_description/meshes/iiwa7/collision/link_0.stl"/>
+          <mesh filename="package://robot_agent_gazebo/models/kuka_with_plate/meshes/iiwa7/visual/link_0.stl"/>
+        </geometry>
+        <material name="Grey"/>
+      </visual>
+      <collision>
+        <origin xyz="0 0 0" rpy="0 0 0"/>
+        <geometry>
+          <mesh filename="package://robot_agent_gazebo/models/kuka_with_plate/meshes/iiwa7/collision/link_0.stl"/>
         </geometry>
         <material name="Grey"/>
@@ -70,5 +70,5 @@
         <origin xyz="0 0 0.0075" rpy="0 0 0"/>
         <geometry>
-          <mesh filename="package://iiwa_description/meshes/iiwa7/visual/link_1.stl"/>
+          <mesh filename="package://robot_agent_gazebo/models/kuka_with_plate/meshes/iiwa7/visual/link_1.stl"/>
         </geometry>
         <material name="Orange"/>
@@ -77,5 +77,5 @@
         <origin xyz="0 0 0.0075" rpy="0 0 0"/>
         <geometry>
-          <mesh filename="package://iiwa_description/meshes/iiwa7/collision/link_1.stl"/>
+          <mesh filename="package://robot_agent_gazebo/models/kuka_with_plate/meshes/iiwa7/collision/link_1.stl"/>
         </geometry>
         <material name="Orange"/>
@@ -104,12 +104,12 @@
         <origin xyz="0 0 0" rpy="0 0 0"/>
         <geometry>
-          <mesh filename="package://iiwa_description/meshes/iiwa7/visual/link_2.stl"/>
-        </geometry>
-        <material name="Orange"/>
-      </visual>
-      <collision>
-        <origin xyz="0 0 0" rpy="0 0 0"/>
-        <geometry>
-          <mesh filename="package://iiwa_description/meshes/iiwa7/collision/link_2.stl"/>
+          <mesh filename="package://robot_agent_gazebo/models/kuka_with_plate/meshes/iiwa7/visual/link_2.stl"/>
+        </geometry>
+        <material name="Orange"/>
+      </visual>
+      <collision>
+        <origin xyz="0 0 0" rpy="0 0 0"/>
+        <geometry>
+          <mesh filename="package://robot_agent_gazebo/models/kuka_with_plate/meshes/iiwa7/collision/link_2.stl"/>
         </geometry>
         <material name="Orange"/>
@@ -138,12 +138,12 @@
         <origin xyz="0 0 -0.026" rpy="0 0 0"/>
         <geometry>
-          <mesh filename="package://iiwa_description/meshes/iiwa7/visual/link_3.stl"/>
-        </geometry>
-        <material name="Orange"/>
-      </visual>
-      <collision>
-        <origin xyz="0 0 -0.026" rpy="0 0 0"/>
-        <geometry>
-          <mesh filename="package://iiwa_description/meshes/iiwa7/collision/link_3.stl"/>
+          <mesh filename="package://robot_agent_gazebo/models/kuka_with_plate/meshes/iiwa7/visual/link_3.stl"/>
+        </geometry>
+        <material name="Orange"/>
+      </visual>
+      <collision>
+        <origin xyz="0 0 -0.026" rpy="0 0 0"/>
+        <geometry>
+          <mesh filename="package://robot_agent_gazebo/models/kuka_with_plate/meshes/iiwa7/collision/link_3.stl"/>
         </geometry>
         <material name="Orange"/>
@@ -172,12 +172,12 @@
         <origin xyz="0 0 0" rpy="0 0 0"/>
         <geometry>
-          <mesh filename="package://iiwa_description/meshes/iiwa7/visual/link_4.stl"/>
-        </geometry>
-        <material name="Orange"/>
-      </visual>
-      <collision>
-        <origin xyz="0 0 0" rpy="0 0 0"/>
-        <geometry>
-          <mesh filename="package://iiwa_description/meshes/iiwa7/collision/link_4.stl"/>
+          <mesh filename="package://robot_agent_gazebo/models/kuka_with_plate/meshes/iiwa7/visual/link_4.stl"/>
+        </geometry>
+        <material name="Orange"/>
+      </visual>
+      <collision>
+        <origin xyz="0 0 0" rpy="0 0 0"/>
+        <geometry>
+          <mesh filename="package://robot_agent_gazebo/models/kuka_with_plate/meshes/iiwa7/collision/link_4.stl"/>
         </geometry>
         <material name="Orange"/>
@@ -206,12 +206,12 @@
         <origin xyz="0 0 -0.026" rpy="0 0 0"/>
         <geometry>
-          <mesh filename="package://iiwa_description/meshes/iiwa7/visual/link_5.stl"/>
-        </geometry>
-        <material name="Orange"/>
-      </visual>
-      <collision>
-        <origin xyz="0 0 -0.026" rpy="0 0 0"/>
-        <geometry>
-          <mesh filename="package://iiwa_description/meshes/iiwa7/collision/link_5.stl"/>
+          <mesh filename="package://robot_agent_gazebo/models/kuka_with_plate/meshes/iiwa7/visual/link_5.stl"/>
+        </geometry>
+        <material name="Orange"/>
+      </visual>
+      <collision>
+        <origin xyz="0 0 -0.026" rpy="0 0 0"/>
+        <geometry>
+          <mesh filename="package://robot_agent_gazebo/models/kuka_with_plate/meshes/iiwa7/collision/link_5.stl"/>
         </geometry>
         <material name="Orange"/>
@@ -240,12 +240,12 @@
         <origin xyz="0 0 0" rpy="0 0 0"/>
         <geometry>
-          <mesh filename="package://iiwa_description/meshes/iiwa7/visual/link_6.stl"/>
-        </geometry>
-        <material name="Orange"/>
-      </visual>
-      <collision>
-        <origin xyz="0 0 0" rpy="0 0 0"/>
-        <geometry>
-          <mesh filename="package://iiwa_description/meshes/iiwa7/collision/link_6.stl"/>
+          <mesh filename="package://robot_agent_gazebo/models/kuka_with_plate/meshes/iiwa7/visual/link_6.stl"/>
+        </geometry>
+        <material name="Orange"/>
+      </visual>
+      <collision>
+        <origin xyz="0 0 0" rpy="0 0 0"/>
+        <geometry>
+          <mesh filename="package://robot_agent_gazebo/models/kuka_with_plate/meshes/iiwa7/collision/link_6.stl"/>
         </geometry>
         <material name="Orange"/>
@@ -274,5 +274,5 @@
         <origin xyz="0 0 -0.0005" rpy="0 0 0"/>
         <geometry>
-          <mesh filename="package://iiwa_description/meshes/iiwa7/visual/link_7.stl"/>
+          <mesh filename="package://robot_agent_gazebo/models/kuka_with_plate/meshes/iiwa7/visual/link_7.stl"/>
         </geometry>
         <material name="Grey"/>
@@ -281,5 +281,5 @@
         <origin xyz="0 0 -0.0005" rpy="0 0 0"/>
         <geometry>
-          <mesh filename="package://iiwa_description/meshes/iiwa7/collision/link_7.stl"/>
+          <mesh filename="package://robot_agent_gazebo/models/kuka_with_plate/meshes/iiwa7/collision/link_7.stl"/>
         </geometry>
         <material name="Grey"/>

File: robot_agent_gazebo/models/kuka_with_plate/urdf/kuka_with_plate.urdf.xacro (robot description, xacro)
@@ -2,8 +2,9 @@
 <robot name="kuka_with_plate" xmlns:xacro="http://www.ros.org/wiki/xacro">
 	<xacro:include filename="iiwa7.urdf.xacro"/>
-	<xacro:include filename="EEplate.urdf.xacro" name="ee_plate" parent="iiwa_link_7" thickness="0.05" radius="0.25">
-		<origin xyz="0 0 0" rpy="0 0 0"/>
-	</xacro:include>
-	<gazebo reference="EEplate_base">
+	<xacro:include filename="EEplate.urdf.xacro"/>
+	<xacro:EEplate parent="iiwa_link_7" name="plate" radius="0.2" thickness="0.04">
+    	<origin xyz="0 0 0" rpy="0 ${pi/2} 0" />
+  	</xacro:EEplate>
+	<gazebo reference="plate_base">
 		<material>Gazebo/Grey</material>
 	</gazebo>
