Commit message: Changed hardware interface back to effort control, replaced trajectory control with individual joint position control

File: robot_agent_gazebo/models/kuka_with_plate/urdf/iiwa7.urdf.xacro (robot description, xacro)
@@ -5,5 +5,5 @@
   <!--Import the lbr iiwa macro -->
   <xacro:include filename="$(find robot_agent_gazebo)/models/kuka_with_plate/urdf/iiwa7.xacro"/>
-  <xacro:arg name="hardware_interface" default="PositionJointInterface"/>
+  <xacro:arg name="hardware_interface" default="EffortJointInterface"/>
   <xacro:arg name="robot_name" default="iiwa"/>
   <xacro:arg name="origin_xyz" default="0 0 0"/>

File: robot_agent_gazebo/models/kuka_with_plate/urdf/iiwa7.xacro (robot description, xacro)
@@ -11,6 +11,6 @@
   <xacro:property name="safety_controller_k_vel" value="2" />
   <xacro:property name="joint_damping" value="0.5" />
-  <xacro:property name="max_effort" value="300"/>
-  <xacro:property name="max_velocity" value="10"/>
+  <xacro:property name="max_effort" value="3000000"/> <!--original values for max effort/vel were 300/10-->
+  <xacro:property name="max_velocity" value="1000"/>
   <xacro:macro name="iiwa7" params="parent hardware_interface robot_name *origin">
     <!--joint between {parent} and link_0-->

File: robot_agent_gazebo/models/kuka_with_plate/urdf/kuka_with_plate.urdf.xacro (robot description, xacro)
@@ -9,5 +9,5 @@
 		<material>Gazebo/Grey</material>
 	</gazebo>
-	<gazebo reference="iiwa_link_0">
+	<!--gazebo reference="iiwa_link_0">
 		<turnGravityOff>true</turnGravityOff>
 	</gazebo>
@@ -32,4 +32,4 @@
 	<gazebo reference="iiwa_link_7">
 		<turnGravityOff>true</turnGravityOff>
-	</gazebo>
+	</gazebo-->
 </robot>
