Commit message: Update iiwa7.xacro
Fixing joint 1 and joint 2 in place at 0 degrees

File: robot_agent_gazebo/models/kuka_with_plate/urdf/iiwa7.xacro (robot description, xacro)
@@ -53,6 +53,6 @@
       <origin xyz="0 0 0.15" rpy="0 0 0"/>
       <axis xyz="0 0 1"/>
-      <limit lower="${-170 * PI / 180}" upper="${170 * PI / 180}"
-             effort="${max_effort}" velocity="${max_velocity}" />
+      <limit lower="0" upper="0"
+             effort="${max_effort}" velocity="${max_velocity}" />     <!-- was previously limit lower="${-170 * PI / 180}" upper="${170 * PI / 180}" -->
       <safety_controller soft_lower_limit="${-168 * PI / 180}"
                          soft_upper_limit="${168 * PI / 180}"
@@ -87,6 +87,6 @@
       <origin xyz="0 0 0.19" rpy="${PI / 2}   0 ${PI}"/>
       <axis xyz="0 0 1"/>
-      <limit lower="${-120 * PI / 180}" upper="${120 * PI / 180}"
-             effort="${max_effort}" velocity="${max_velocity}" />
+      <limit lower="0" upper="0"
+             effort="${max_effort}" velocity="${max_velocity}" />    <!-- was previously limit lower="${-120 * PI / 180}" upper="${120 * PI / 180}" -->
       <safety_controller soft_lower_limit="${-118 * PI / 180}"
                          soft_upper_limit="${118 * PI / 180}"
